File: Templates/EXT_Connectors.kicad_sch (KiCad schematic)
At the start: 11 parts, among them J1 DC-005, J3 Micro_SD_Card, J9 OK-14F024-04

Commit message: update: 修复库文件缺失
Parts:
- removed BAT1: CR2032, DuRuofu_Connector:BAT-TH_BS-2-1, symbol EXT_Connectors:CR2032-2-1
- added BAT2: CR2032, EXT_Connectors_THT:BAT-TH_BS-2-1, symbol EXT_Connectors:CR2032
Changed lines of the file:
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@@
+	)
+	(symbol
+		(lib_id "EXT_Connectors:CR2032")
+		(at 40.64 38.1 0)
+		(unit 1)
+		(exclude_from_sim no)
+		(in_bom yes)
+		(on_board yes)
+		(dnp no)
+		(fields_autoplaced yes)
+		(property "Reference" "BAT2"
+			(at 40.005 30.48 0)
+			(effects
+				(font
+					(size 1.27 1.27)
+				)
+			)
+		)
+		(property "Value" "CR2032"
+			(at 40.005 33.02 0)
+			(effects
+				(font
+					(size 1.27 1.27)
+				)
+			)
+		)
+		(property "Footprint" "EXT_Connectors_THT:BAT-TH_BS-2-1"
+			(at 40.894 33.02 0)
+			(effects
+				(font
+					(size 1.27 1.27)
+				)
+				(hide yes)
+			)
+		)
+		(property "Datasheet" ""
+			(at 40.894 33.02 0)
+			(effects
+				(font
+					(size 1.27 1.27)
+				)
+				(hide yes)
+			)
+		)
+		(property "Description" ""
+			(at 40.894 33.02 0)
+			(effects
+				(font
+					(size 1.27 1.27)
+				)
+				(hide yes)
+			)
+		)
+		(pin "1"
+		)
+		(pin "2"
+		)
+		(instances
+			(project ""
+				(path "/15ae7a0d-a53d-4804-b6bf-a747840a1ecc/580d79ab-0767-4e48-865a-215fd5c8ce7b"
+					(reference "BAT2")
+					(unit 1)
+				)
+			)
+		)
 	)
 	(symbol
@@
 					(unit 1)
 				)
-			)
-		)
-	)
-	(symbol
-		(lib_id "EXT_Connectors:CR2032-2-1")
-		(at 46.99 38.1 0)
-		(unit 1)
-		(exclude_from_sim no)
-		(in_bom yes)
-		(on_board yes)
-		(dnp no)
-		(fields_autoplaced yes)
-		(property "Reference" "BAT1"
-			(at 46.355 30.48 0)
-			(effects
-				(font
-					(size 1.27 1.27)
-				)
-			)
-		)
-		(property "Value" "CR2032"
-			(at 46.355 33.02 0)
-			(effects
-				(font
-					(size 1.27 1.27)
-				)
-			)
-		)
-		(property "Footprint" "DuRuofu_Connector:BAT-TH_BS-2-1"
-			(at 47.244 33.02 0)
-			(effects
-				(font
-					(size 1.27 1.27)
-				)
-				(hide yes)
-			)
-		)
-		(property "Datasheet" ""
-			(at 47.244 33.02 0)
-			(effects
-				(font
-					(size 1.27 1.27)
-				)
-				(hide yes)
-			)
-		)
-		(property "Description" ""
-			(at 47.244 33.02 0)
-			(effects
-				(font
-					(size 1.27 1.27)
-				)
-				(hide yes)
-			)
-		)
-		(pin "2"
-		)
-		(pin "1"
-		)
-		(instances
-			(project ""
-				(path "/15ae7a0d-a53d-4804-b6bf-a747840a1ecc/580d79ab-0767-4e48-865a-215fd5c8ce7b"
-					(reference "BAT1")
-					(unit 1)
-				)
