File: Templates/EXT_Modules.kicad_sch (KiCad schematic)
At the start: 4 parts

Commit message: update: 添加器件-合宙ESP32S3开发板
Parts:
- added U28: ~, EXT_Modules:合宙ESP32C3开发板-DIP&SMT, symbol EXT_Modules:合宙ESP32C3开发板-DIP&SMT
Changed lines of the file:
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@@
+	)
+	(symbol
+		(lib_id "EXT_Modules:合宙ESP32C3开发板-DIP&SMT")
+		(at 196.85 45.72 0)
+		(unit 1)
+		(exclude_from_sim no)
+		(in_bom yes)
+		(on_board yes)
+		(dnp no)
+		(fields_autoplaced yes)
+		(property "Reference" "U28"
+			(at 215.9 21.59 0)
+			(effects
+				(font
+					(size 1.27 1.27)
+				)
+			)
+		)
+		(property "Value" "~"
+			(at 215.9 24.13 0)
+			(effects
+				(font
+					(size 1.27 1.27)
+				)
+			)
+		)
+		(property "Footprint" "EXT_Modules:合宙ESP32C3开发板-DIP&SMT"
+			(at 196.85 45.72 0)
+			(effects
+				(font
+					(size 1.27 1.27)
+				)
+				(hide yes)
+			)
+		)
+		(property "Datasheet" ""
+			(at 196.85 45.72 0)
+			(effects
+				(font
+					(size 1.27 1.27)
+				)
+				(hide yes)
+			)
+		)
+		(property "Description" ""
+			(at 196.85 45.72 0)
+			(effects
+				(font
+					(size 1.27 1.27)
+				)
+				(hide yes)
+			)
+		)
+		(pin "32"
+		)
+		(pin "22"
+		)
+		(pin "23"
+		)
+		(pin "19"
+		)
+		(pin "13"
+		)
+		(pin "25"
+		)
+		(pin "3"
+		)
+		(pin "6"
+		)
+		(pin "7"
+		)
+		(pin "11"
+		)
+		(pin "16"
+		)
+		(pin "24"
+		)
+		(pin "28"
+		)
+		(pin "29"
+		)
+		(pin "10"
+		)
+		(pin "1"
+		)
+		(pin "15"
+		)
+		(pin "30"
+		)
+		(pin "31"
+		)
+		(pin "8"
+		)
+		(pin "27"
+		)
+		(pin "2"
+		)
+		(pin "21"
+		)
+		(pin "5"
+		)
+		(pin "12"
+		)
+		(pin "14"
+		)
+		(pin "4"
+		)
+		(pin "18"
+		)
+		(pin "20"
+		)
+		(pin "26"
+		)
+		(pin "17"
+		)
+		(pin "9"
+		)
+		(instances
+			(project ""
+				(path "/15ae7a0d-a53d-4804-b6bf-a747840a1ecc/7c4262aa-b448-4bef-a6bf-9d88d3bd0d6e"
+					(reference "U28")
+					(unit 1)
+				)
+			)
+		)
 	)
 	(symbol
