File: Templates/Templates.kicad_sch (KiCad schematic)
At the start: 0 parts

Commit message: update:添加文件
Other:
- added sheet EXT_Connectors (EXT_Connectors.kicad_sch)
- added sheet EXT_ICs (EXT_ICs.kicad_sch)
- added sheet EXT_Modules (EXT_Modules.kicad_sch)
- added sheet EXT_Other (EXT_Other.kicad_sch)
- added sheet EXT_Passive (EXT_Passive.kicad_sch)
- added sheet EXT_Switch (EXT_Switch.kicad_sch)
